File: DinoEDA/testEDA/testEDA.kicad_sch (KiCad schematic)
At the start: 9 parts, among them U1 NE555D

Commit message: Still figuring things out
Parts:
- C1, C2: footprint (none) -> Capacitor_SMD:CP_Elec_3x5.3
- D1, D2: footprint (none) -> Diode_SMD:D_0201_0603Metric
- D3: footprint (none) -> Connector_Audio:Jack_3.5mm_CUI_SJ-3523-SMT_Horizontal
- POT1: footprint (none) -> Potentiometer_THT:Potentiometer_ACP_CA6-H2,5_Horizontal
- R1, R2: footprint (none) -> Resistor_SMD:R_0201_0603Metric
Changed lines of the file:
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@@
     (property "Reference" "D1" (id 0) (at 123.19 72.39 0))
     (property "Value" "DIODE" (id 1) (at 119.38 71.12 0))
-    (property "Footprint" "" (id 2) (at 124.46 68.58 0)
+    (property "Footprint" "Diode_SMD:D_0201_0603Metric" (id 2) (at 124.46 68.58 0)
       (effects (font (size 1.27 1.27)) hide)
     )
@@
     (property "Reference" "C1" (id 0) (at 85.09 83.82 90))
     (property "Value" "100nF" (id 1) (at 85.09 86.36 90))
-    (property "Footprint" "" (id 2) (at 88.9 90.4748 0)
+    (property "Footprint" "Capacitor_SMD:CP_Elec_3x5.3" (id 2) (at 88.9 90.4748 0)
       (effects (font (size 1.27 1.27)) hide)
     )
@@
       (effects (font (size 1.27 1.27)) (justify right))
     )
-    (property "Footprint" "" (id 2) (at 193.04 95.25 0)
+    (property "Footprint" "Connector_Audio:Jack_3.5mm_CUI_SJ-3523-SMT_Horizontal" (id 2) (at 193.04 95.25 0)
       (effects (font (size 1.27 1.27)) hide)
     )
@@
       (effects (font (size 1.27 1.27)) (justify left))
     )
-    (property "Footprint" "" (id 2) (at 101.2952 124.46 0)
+    (property "Footprint" "Capacitor_SMD:CP_Elec_3x5.3" (id 2) (at 101.2952 124.46 0)
       (effects (font (size 1.27 1.27)) hide)
     )
@@
     (property "Reference" "R2" (id 0) (at 154.94 88.9 90))
     (property "Value" "15" (id 1) (at 158.75 88.9 90))
-    (property "Footprint" "" (id 2) (at 156.21 93.218 90)
+    (property "Footprint" "Resistor_SMD:R_0201_0603Metric" (id 2) (at 156.21 93.218 90)
       (effects (font (size 1.27 1.27)) hide)
     )
@@
     (property "Reference" "D2" (id 0) (at 123.19 80.01 0))
     (property "Value" "DIODE" (id 1) (at 119.38 78.74 0))
-    (property "Footprint" "" (id 2) (at 124.46 76.2 0)
+    (property "Footprint" "Diode_SMD:D_0201_0603Metric" (id 2) (at 124.46 76.2 0)
       (effects (font (size 1.27 1.27)) hide)
     )
@@
       (effects (font (size 1.27 1.27)) (justify left))
     )
-    (property "Footprint" "" (id 2) (at 137.922 81.28 90)
+    (property "Footprint" "Resistor_SMD:R_0201_0603Metric" (id 2) (at 137.922 81.28 90)
       (effects (font (size 1.27 1.27)) hide)
     )
@@
       (effects (font (size 1.27 1.27)) (justify right))
     )
-    (property "Footprint" "" (id 2) (at 107.95 72.39 0)
+    (property "Footprint" "Potentiometer_THT:Potentiometer_ACP_CA6-H2,5_Horizontal" (id 2) (at 107.95 72.39 0)
       (effects (font (size 1.27 1.27)) hide)
     )
@@
     )
     (path "/75b20854-8775-4afd-95f6-872ef54c14cb"
-      (reference "C1") (unit 1) (value "100nF") (footprint "")
+      (reference "C1") (unit 1) (value "100nF") (footprint "Capacitor_SMD:CP_Elec_3x5.3")
     )
     (path "/989350e0-5184-4598-b17e-fb5ac33086e8"
-      (reference "C2") (unit 1) (value "10nF") (footprint "")
+      (reference "C2") (unit 1) (value "10nF") (footprint "Capacitor_SMD:CP_Elec_3x5.3")
     )
     (path "/474eadca-e236-4182-98a1-1f11b6a12eb1"
-      (reference "D1") (unit 1) (value "DIODE") (footprint "")
+      (reference "D1") (unit 1) (value "DIODE") (footprint "Diode_SMD:D_0201_0603Metric")
     )
     (path "/a4cf543e-6694-4d62-875a-a7568853edbc"
-      (reference "D2") (unit 1) (value "DIODE") (footprint "")
+      (reference "D2") (unit 1) (value "DIODE") (footprint "Diode_SMD:D_0201_0603Metric")
     )
     (path "/8888e6d6-ec4f-4e8b-bcc5-2b96272ea0ac"
-      (reference "D3") (unit 1) (value "LED_Series") (footprint "")
+      (reference "D3") (unit 1) (value "LED_Series") (footprint "Connector_Audio:Jack_3.5mm_CUI_SJ-3523-SMT_Horizontal")
     )
     (path "/f70eae9a-3f70-493d-88a4-a710368f0274"
-      (reference "POT1") (unit 1) (value "10K") (footprint "")
+      (reference "POT1") (unit 1) (value "10K") (footprint "Potentiometer_THT:Potentiometer_ACP_CA6-H2,5_Horizontal")
     )
     (path "/e83477c6-7ad0-4d17-9d4d-8572e5083486"
-      (reference "R1") (unit 1) (value "120") (footprint "")
+      (reference "R1") (unit 1) (value "120") (footprint "Resistor_SMD:R_0201_0603Metric")
     )
     (path "/a365a6a1-7367-4c8c-a245-014801e16d01"
-      (reference "R2") (unit 1) (value "15") (footprint "")
+      (reference "R2") (unit 1) (value "15") (footprint "Resistor_SMD:R_0201_0603Metric")
     )
     (path "/aba1abbf-b9d4-4e20-b19c-207d43ae6497"
